Commit message: feat: updated abluo 1 description

File: abluo_urdf_1/urdf/abluo_urdf_1.urdf (robot description, URDF)
Before this commit: robot abluo_urdf_1, 2 links, 1 joints
Links:
- removed link linear_actuator
- added link bin, mass 0.26632; collision mesh filename=package://abluo_urdf_1/meshes/bin.STL; visual mesh filename=package://abluo_urdf_1/meshes/bin.STL
- added link refill, mass 0.48444; collision mesh filename=package://abluo_urdf_1/meshes/refill.STL; visual mesh filename=package://abluo_urdf_1/meshes/refill.STL
- added link robot_arm_mount, mass 0.42315; collision mesh filename=package://abluo_urdf_1/meshes/robot_arm_mount.STL; visual mesh filename=package://abluo_urdf_1/meshes/robot_arm_mount.STL
- added link tool_holder, mass 0.1248; collision mesh filename=package://abluo_urdf_1/meshes/tool_holder.STL; visual mesh filename=package://abluo_urdf_1/meshes/tool_holder.STL
- link base_link: mass 14.2555803950512 -> 13.1202235524193
Joints:
- removed joint linear_actuator_to_trolley
- added joint bin_to_trolley: type fixed, parent base_link, child bin, origin xyz=0.41232 0.78622 0.051806 rpy=0 0 0, axis 0 0 0
- added joint refill_to_trolley: type fixed, parent base_link, child refill, origin xyz=0.23641 0.73898 0.11878 rpy=0 0 0, axis 0 0 0
- added joint robot_arm_mount_to_actuator: type prismatic, parent base_link, child robot_arm_mount, origin xyz=0.30617 0.70397 0.49087 rpy=0 0 0, axis 0 0 1, limit lower=-0.2 upper=0.2 effort=0 velocity=0
- added joint tool_holder_to_trolley: type fixed, parent base_link, child tool_holder, origin xyz=0.47532 0.67022 0.32681 rpy=0 0 0, axis 0 0 0
