Commit message: fix: moved aligner on trolley to match real robot

File: arm_plus_base_description/urdf/abluo_urdf_1.xacro (robot description, xacro)
@@ -50,5 +50,5 @@
   </link>
   <joint name="tool_holder_to_trolley" type="fixed">
-    <origin xyz="0.47532 0.67022 0.32681" rpy="0 0 0" />
+    <origin xyz="0.47032 0.67022 0.33281" rpy="0 0 0" />
     <parent link="base_link" />
     <child link="tool_holder" />
@@ -138,5 +138,5 @@
     <child link="robot_arm_mount" />
     <axis xyz="0 0 1" />
-    <limit lower="-0.2" upper="0.18" effort="100000" velocity="0.03" />
+    <limit lower="-0.2" upper="0.16" effort="100000" velocity="0.0235" />
   </joint>
 </robot>
