Commit message: enhancement: abluo_moveit_config updated to match real robot

File: descriptions/arm_plus_base_description/urdf/arm_plus_base.gazebo.xacro (robot description, xacro)
@@ -4,8 +4,8 @@
         <type>transmission_interface/SimpleTransmission</type>
         <joint name="joint2_to_joint1">
-            <hardwareInterface>hardware_interface/EffortJointInterface</hardwareInterface>
+            <hardwareInterface>hardware_interface/PositionJointInterface</hardwareInterface>
         </joint>
         <actuator name="joint2_to_joint1_motor">
-            <hardwareInterface>hardware_interface/EffortJointInterface</hardwareInterface>
+            <hardwareInterface>hardware_interface/PositionJointInterface</hardwareInterface>
             <mechanicalReduction>1</mechanicalReduction>
         </actuator>
@@ -14,8 +14,8 @@
         <type>transmission_interface/SimpleTransmission</type>
         <joint name="joint3_to_joint2">
-            <hardwareInterface>hardware_interface/EffortJointInterface</hardwareInterface>
+            <hardwareInterface>hardware_interface/PositionJointInterface</hardwareInterface>
         </joint>
         <actuator name="joint3_to_joint2_motor">
-            <hardwareInterface>hardware_interface/EffortJointInterface</hardwareInterface>
+            <hardwareInterface>hardware_interface/PositionJointInterface</hardwareInterface>
             <mechanicalReduction>1</mechanicalReduction>
         </actuator>
@@ -24,8 +24,8 @@
         <type>transmission_interface/SimpleTransmission</type>
         <joint name="joint4_to_joint3">
-            <hardwareInterface>hardware_interface/EffortJointInterface</hardwareInterface>
+            <hardwareInterface>hardware_interface/PositionJointInterface</hardwareInterface>
         </joint>
         <actuator name="joint4_to_joint3_motor">
-            <hardwareInterface>hardware_interface/EffortJointInterface</hardwareInterface>
+            <hardwareInterface>hardware_interface/PositionJointInterface</hardwareInterface>
             <mechanicalReduction>1</mechanicalReduction>
         </actuator>
@@ -34,8 +34,8 @@
         <type>transmission_interface/SimpleTransmission</type>
         <joint name="joint5_to_joint4">
-            <hardwareInterface>hardware_interface/EffortJointInterface</hardwareInterface>
+            <hardwareInterface>hardware_interface/PositionJointInterface</hardwareInterface>
         </joint>
         <actuator name="joint5_to_joint4_motor">
-            <hardwareInterface>hardware_interface/EffortJointInterface</hardwareInterface>
+            <hardwareInterface>hardware_interface/PositionJointInterface</hardwareInterface>
             <mechanicalReduction>1</mechanicalReduction>
         </actuator>
@@ -44,8 +44,8 @@
         <type>transmission_interface/SimpleTransmission</type>
         <joint name="joint6_to_joint5">
-            <hardwareInterface>hardware_interface/EffortJointInterface</hardwareInterface>
+            <hardwareInterface>hardware_interface/PositionJointInterface</hardwareInterface>
         </joint>
         <actuator name="joint6_to_joint5_motor">
-            <hardwareInterface>hardware_interface/EffortJointInterface</hardwareInterface>
+            <hardwareInterface>hardware_interface/PositionJointInterface</hardwareInterface>
             <mechanicalReduction>1</mechanicalReduction>
         </actuator>
@@ -54,8 +54,8 @@
         <type>transmission_interface/SimpleTransmission</type>
         <joint name="joint6output_to_joint6">
-            <hardwareInterface>hardware_interface/EffortJointInterface</hardwareInterface>
+            <hardwareInterface>hardware_interface/PositionJointInterface</hardwareInterface>
         </joint>
         <actuator name="joint6output_to_joint6_motor">
-            <hardwareInterface>hardware_interface/EffortJointInterface</hardwareInterface>
+            <hardwareInterface>hardware_interface/PositionJointInterface</hardwareInterface>
             <mechanicalReduction>1</mechanicalReduction>
         </actuator>
@@ -64,8 +64,8 @@
         <type>transmission_interface/SimpleTransmission</type>
         <joint name="robot_arm_mount_to_actuator">
-            <hardwareInterface>hardware_interface/EffortJointInterface</hardwareInterface>
+            <hardwareInterface>hardware_interface/PositionJointInterface</hardwareInterface>
         </joint>
         <actuator name="robot_arm_mount_to_actuator_motor">
-            <hardwareInterface>hardware_interface/EffortJointInterface</hardwareInterface>
+            <hardwareInterface>hardware_interface/PositionJointInterface</hardwareInterface>
             <mechanicalReduction>1</mechanicalReduction>
         </actuator>

File: descriptions/arm_plus_base_description/urdf/arm_plus_base.urdf.xacro (robot description, xacro)
@@ -11,5 +11,5 @@
        <!-- include gazebo transmissions -->
        <xacro:include filename="$(find arm_plus_base_description)/urdf/arm_plus_base.gazebo.xacro"/>
-      <xacro:mycobot_pro_robot_macro camera_sensor="$(arg camera_sensor)" attach_to="$(arg attach_to)" xyz="0 0.015 0" rpy="-1.5707 -1.5707 0"/>
+      <xacro:mycobot_pro_robot_macro camera_sensor="$(arg camera_sensor)" attach_to="$(arg attach_to)" xyz="0 0.015 0" rpy="-1.5707 1.5707 0"/>
   </xacro:macro>
   <xacro:base_arm_macro/>

File: descriptions/arm_plus_base_description/urdf/mycobot_robot_macro.xacro (robot description, xacro)
@@ -17,5 +17,5 @@
       <parent link="link6"/>
       <child link="brush_swapping_stick_link"/>>
-      <origin xyz="0 0 0" rpy="-1.57 0 0"/>
+      <origin xyz="0 0 0" rpy="-1.57 0 1.57"/>
     </joint>
   </xacro:macro>
