Commit message: mycobot_alone actuating

File: descriptions/arm_plus_base_description/urdf/abluo_urdf_1.xacro (robot description, xacro)
@@ -133,5 +133,5 @@
     </collision>
   </link>
-  <joint name="robot_arm_mount_to_actuator" type="prismatic">
+  <joint name="robot_arm_mount_to_actuator" type="fixed">
     <origin xyz="0.30617 0.70397 0.49087" rpy="0 0 0" />
     <parent link="base_link" />
